File: kicad_pendant/kicad_pendant.kicad_pcb (KiCad board)
At the start: 2 copper layers, 71.1 x 95.2 mm, 39 parts, among them J1 Conn_01x12_Female, J2 Conn_01x12_Female, SW1 SW_Push, SW2 SW_Push, SW3 SW_Push, SW4 SW_Push, SW5 SW_Push, SW6 SW_Push, SW7 SW_Push, SW8 SW_Push, SW9 SW_Push

Commit message: Board design V1
Parts:
- added ?: , custom:logo_plane, B.Cu at (166.4, 54.6)
- added G***: LOGO, custom:plane_3, F.Cu at (137.2, 27.9)
- added REF**: OSHW-Logo2_14.6x12mm_SilkScreen, Symbol:OSHW-Logo2_14.6x12mm_SilkScreen, F.Cu at (158.8, 29.2)
- added REF**: OSHW-Logo2_14.6x12mm_SilkScreen, Symbol:OSHW-Logo2_14.6x12mm_SilkScreen, B.Cu at (158.8, 29.2)
Other:
- board text added: "Creative Commons BY-SA 4.0"
- board text added: "TTGO T-Display ESP32"
- board text added: "TallyBandit.com"
- board text added: "Wireless CNC Pendant"

Commit message: Adding modified kicad board
Parts:
- SW1, SW2, SW3, SW4, SW5, SW6, SW7, SW8, SW9: footprint Button_Switch_Keyboard:SW_Cherry_MX_1.00u_PCB -> custom:SW_Cherry_MX_1.00u_PCB

Commit message: Undo PCB changes
Parts:
- SW1, SW2, SW3, SW4, SW5, SW6, SW7, SW8, SW9: footprint custom:SW_Cherry_MX_1.00u_PCB -> Button_Switch_Keyboard:SW_Cherry_MX_1.00u_PCB
